File: hardware/laserRangerExploration/laserRangerExploration.kicad_pcb (KiCad board)
At the start: 2 copper layers, 25.2 x 25.2 mm, 2 parts

Commit message: small pcb update
Parts:
- N2: value 20181108 -> 20190606
Changed lines of the file:
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@@
-(kicad_pcb (version 20171130) (host pcbnew 5.0.2-bee76a0~70~ubuntu18.04.1)
+(kicad_pcb (version 20171130) (host pcbnew 5.1.2-f72e74a~84~ubuntu18.04.1)
   (general
     (thickness 1.6)
@@
     (zone_45_only no)
     (trace_min 0.1524)
-    (segment_width 0.2)
-    (edge_width 0.15)
     (via_size 0.381)
     (via_drill 0.254)
@@
     (uvia_min_size 0.381)
     (uvia_min_drill 0.254)
+    (edge_width 0.15)
+    (segment_width 0.2)
     (pcb_text_width 0.3)
     (pcb_text_size 1.5 1.5)
@@
       (effects (font (size 1 1) (thickness 0.15)))
     )
-    (fp_text value 20181108 (at -0.4 -0.1) (layer F.SilkS)
-      (effects (font (size 1 1) (thickness 0.15)))
-    )
+    (fp_text value 20190606 (at -0.4 -0.1) (layer F.SilkS)
+      (effects (font (size 1 1) (thickness 0.15)))
+    )
